File: board/WiFiModem.kicad_pcb (KiCad board)
At the start: 2 copper layers, 88.9 x 61 mm, 46 parts, among them J1 DB9_Female, J2 DB25_Female, J3 Barrel_Jack_Switch, J4 PRG, SW1 SW_Push, SW2 SW_Push, U1 ESP-12E, U2 LM7805_TO220, U3 MAX232, U4 LT1117-3.3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

Commit message: Added picture of completed boarD
Routing:
- net DCD: track 166.6 -> 165.3 mm
Changed lines of the file:
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@@
     (property "Sheetname" "")
     (attr through_hole)
-    (fp_text reference "J1" (at -5.54 -3.7 90) (layer "F.SilkS")
+    (fp_text reference "J1" (at -5.595 -3.5 90) (layer "F.SilkS")
       (effects (font (size 1 1) (thickness 0.15)))
     )
@@
   (segment (start 125.25 125.45) (end 126.17 124.53) (width 0.35) (layer "F.Cu") (net 20))
   (via (at 125.25 125.45) (size 0.8) (drill 0.4) (layers "F.Cu" "B.Cu") (net 20))
+  (segment (start 155.12 103.95) (end 154.765 104.305) (width 0.35) (layer "B.Cu") (net 20))
   (segment (start 124.206 113.98) (end 125.02 113.98) (width 0.35) (layer "B.Cu") (net 20))
-  (segment (start 75.12 98.75) (end 77.48 96.39) (width 0.35) (layer "B.Cu") (net 20))
-  (segment (start 77.48 96.39) (end 82.52 96.39) (width 0.35) (layer "B.Cu") (net 20))
   (segment (start 154.765 104.305) (end 153.67 104.305) (width 0.35) (layer "B.Cu") (net 20))
+  (segment (start 75.12 98.75) (end 77.48 96.39) (width 0.35) (layer "B.Cu") (net 20))
   (segment (start 158.35 108.98) (end 158.35 104.74) (width 0.35) (layer "B.Cu") (net 20))
-  (segment (start 75.12 124.52) (end 75.12 98.75) (width 0.35) (layer "B.Cu") (net 20))
+  (segment (start 158.91 122.26) (end 158.91 109.54) (width 0.35) (layer "B.Cu") (net 20))
   (segment (start 125.2 125.5) (end 125.2 125.95) (width 0.35) (layer "B.Cu") (net 20))
   (segment (start 125.02 113.98) (end 126.492 112.508) (width 0.35) (layer "B.Cu") (net 20))
   (segment (start 126.492 109.22) (end 129.2 106.512) (width 0.35) (layer "B.Cu") (net 20))
-  (segment (start 125.2 125.95) (end 154.24 125.95) (width 0.35) (layer "B.Cu") (net 20))
-  (segment (start 154.24 125.95) (end 158.91 121.28) (width 0.35) (layer "B.Cu") (net 20))
-  (segment (start 158.91 121.28) (end 158.91 109.54) (width 0.35) (layer "B.Cu") (net 20))
-  (segment (start 155.12 103.95) (end 154.765 104.305) (width 0.35) (layer "B.Cu") (net 20))
+  (segment (start 158.91 109.54) (end 158.35 108.98) (width 0.35) (layer "B.Cu") (net 20))
   (segment (start 125.25 125.45) (end 125.2 125.5) (width 0.35) (layer "B.Cu") (net 20))
-  (segment (start 76.55 125.95) (end 75.12 124.52) (width 0.35) (layer "B.Cu") (net 20))
+  (segment (start 79.7 125.95) (end 75.12 121.37) (width 0.35) (layer "B.Cu") (net 20))
+  (segment (start 77.48 96.39) (end 82.52 96.39) (width 0.35) (layer "B.Cu") (net 20))
   (segment (start 126.492 112.508) (end 126.492 109.22) (width 0.35) (layer "B.Cu") (net 20))
-  (segment (start 125.2 125.95) (end 76.55 125.95) (width 0.35) (layer "B.Cu") (net 20))
-  (segment (start 158.91 109.54) (end 158.35 108.98) (width 0.35) (layer "B.Cu") (net 20))
+  (segment (start 125.2 125.95) (end 155.22 125.95) (width 0.35) (layer "B.Cu") (net 20))
+  (segment (start 125.2 125.95) (end 79.7 125.95) (width 0.35) (layer "B.Cu") (net 20))
+  (segment (start 75.12 121.37) (end 75.12 98.75) (width 0.35) (layer "B.Cu") (net 20))
+  (segment (start 155.22 125.95) (end 158.91 122.26) (width 0.35) (layer "B.Cu") (net 20))
   (segment (start 158.35 104.74) (end 157.56 103.95) (width 0.35) (layer "B.Cu") (net 20))
   (segment (start 129.2 106.512) (end 129.2 105.9) (width 0.35) (layer "B.Cu") (net 20))
